Commit message: organized /vision, refactored files for UR30

File: vision/urdf/ur30_robotiq_realsense.urdf.xacro (robot description, xacro)
@@ -14,6 +14,8 @@
   </xacro:ur_robot>
   <!-- Instantiate Robotiq gripper macro attaching base to tool0 -->
-  <xacro:robotiq_gripper name="RobotiqGripper" prefix="" parent="tool0">
-    <origin xyz="0 0 0" rpy="0 0 0"/>
+  <xacro:robotiq_gripper name="RobotiqGripper" prefix="" parent="tool0"
+                         include_ros2_control="false">
+    <!-- align Robotiq flange with the UR wrist -->
+    <origin xyz="0 0 0" rpy="0 0 ${pi/2}"/>
   </xacro:robotiq_gripper>
   <!-- Camera mount attached to new base link name -->
@@ -39,5 +41,5 @@
     <sensor type="depth" name="realsense_d435i"><update_rate>30</update_rate><camera><horizontal_fov>1.204</horizontal_fov><image><width>848</width><height>480</height><format>R8G8B8</format></image><clip><near>0.28</near><far>3.0</far></clip><noise><type>gaussian</type><mean>0.0</mean><stddev>0.02</stddev></noise></camera><plugin name="camera_plugin" filename="libgazebo_ros_camera.so"><ros><namespace>/</namespace><remapping>~/image_raw:=camera/color/image_raw</remapping><remapping>~/image_depth:=camera/depth/image_rect_raw</remapping><remapping>~/camera_info:=camera/color/camera_info</remapping><remapping>~/camera_info_depth:=camera/depth/camera_info</remapping><remapping>~/points:=camera/depth/color/points</remapping></ros><camera_name>camera</camera_name><frame_name>camera_color_optical_frame</frame_name><hack_baseline>0.0</hack_baseline><min_depth>0.28</min_depth><max_depth>3.0</max_depth></plugin></sensor>
   </gazebo>
-  <!-- Reuse ros2_control from included gripper macro & add arm controllers file -->
+  <!-- Single ros2_control block drives arm and gripper joints in Gazebo -->
   <gazebo><plugin filename="libgazebo_ros2_control.so" name="gazebo_ros2_control"><robot_sim_type>gazebo_ros2_control/GazeboSystem</robot_sim_type><parameters>$(find unified_vision_system)/config/simulation_controllers.yaml</parameters></plugin></gazebo>
   <ros2_control name="GazeboSystem" type="system">
@@ -87,7 +89,72 @@
     </joint>
   </ros2_control>
+  <!-- Gazebo physics parameters for gripper joints to prevent oscillation -->
+  <!-- Main actuated joint -->
   <gazebo reference="robotiq_85_left_knuckle_joint">
+    <implicitSpringDamper>true</implicitSpringDamper>
+    <springStiffness>0.0</springStiffness>
+    <springReference>0.0</springReference>
+    <dampingFactor>10.0</dampingFactor>
+    <kp>1000000.0</kp>
+    <kd>100.0</kd>
     <cfm>0.0</cfm>
     <erp>0.9</erp>
+    <mu1>1.0</mu1>
+    <mu2>1.0</mu2>
+  </gazebo>
+  <!-- Mimic joint (right knuckle) -->
+  <gazebo reference="robotiq_85_right_knuckle_joint">
+    <implicitSpringDamper>true</implicitSpringDamper>
+    <springStiffness>0.0</springStiffness>
+    <springReference>0.0</springReference>
+    <dampingFactor>10.0</dampingFactor>
+    <kp>1000000.0</kp>
+    <kd>100.0</kd>
+    <cfm>0.0</cfm>
+    <erp>0.9</erp>
+    <mu1>1.0</mu1>
+    <mu2>1.0</mu2>
+  </gazebo>
+  <!-- Inner knuckle joints (continuous, need heavy damping) -->
+  <gazebo reference="robotiq_85_left_inner_knuckle_joint">
+    <implicitSpringDamper>true</implicitSpringDamper>
+    <dampingFactor>50.0</dampingFactor>
+    <kp>1000000.0</kp>
+    <kd>100.0</kd>
+    <cfm>0.0</cfm>
+    <erp>0.9</erp>
+    <mu1>1.0</mu1>
+    <mu2>1.0</mu2>
+  </gazebo>
+  <gazebo reference="robotiq_85_right_inner_knuckle_joint">
+    <implicitSpringDamper>true</implicitSpringDamper>
+    <dampingFactor>50.0</dampingFactor>
+    <kp>1000000.0</kp>
+    <kd>100.0</kd>
+    <cfm>0.0</cfm>
+    <erp>0.9</erp>
+    <mu1>1.0</mu1>
+    <mu2>1.0</mu2>
+  </gazebo>
+  <!-- Finger tip joints -->
+  <gazebo reference="robotiq_85_left_finger_tip_joint">
+    <implicitSpringDamper>true</implicitSpringDamper>
+    <dampingFactor>30.0</dampingFactor>
+    <kp>1000000.0</kp>
+    <kd>100.0</kd>
+    <cfm>0.0</cfm>
+    <erp>0.9</erp>
+    <mu1>1.0</mu1>
+    <mu2>1.0</mu2>
+  </gazebo>
+  <gazebo reference="robotiq_85_right_finger_tip_joint">
+    <implicitSpringDamper>true</implicitSpringDamper>
+    <dampingFactor>30.0</dampingFactor>
+    <kp>1000000.0</kp>
+    <kd>100.0</kd>
+    <cfm>0.0</cfm>
+    <erp>0.9</erp>
+    <mu1>1.0</mu1>
+    <mu2>1.0</mu2>
   </gazebo>
 </robot>

Commit message: realsense camera configured, UR30 kinematics configured, Workspace validator configured - beginning test scenario configuration

File: vision/urdf/ur30_robotiq_realsense.urdf.xacro (robot description, xacro)
@@ -27,5 +27,5 @@
   </joint>
   <link name="camera_link"><inertial><origin xyz="0 0 0" rpy="0 0 0"/><mass value="0.072"/><inertia ixx="1e-05" ixy="0" ixz="0" iyy="1e-05" iyz="0" izz="1e-05"/></inertial><visual><origin xyz="0 0 0" rpy="0 0 0"/><geometry><box size="0.025 0.09 0.025"/></geometry><material name="black"><color rgba="0.1 0.1 0.1 1"/></material></visual><collision><origin xyz="0 0 0" rpy="0 0 0"/><geometry><box size="0.025 0.09 0.025"/></geometry></collision></link>
-  <joint name="camera_joint" type="fixed"><parent link="camera_mount_link"/><child link="camera_link"/><origin xyz="0 0 0.015" rpy="0 0 0"/></joint>
+  <joint name="camera_joint" type="fixed"><parent link="camera_mount_link"/><child link="camera_link"/><origin xyz="0 0 0.015" rpy="${-pi/2} ${-pi/2} 0"/></joint>
   <link name="camera_color_frame"/>
   <joint name="camera_color_joint" type="fixed"><parent link="camera_link"/><child link="camera_color_frame"/><origin xyz="0 0 0" rpy="0 0 0"/></joint>

File: vision/urdf/ur30_simple_gripper_realsense.urdf.xacro (robot description, xacro)
@@ -86,5 +86,5 @@
     <parent link="camera_mount_link"/>
     <child link="camera_link"/>
-    <origin xyz="0 0 0.015" rpy="0 0 0"/>
+    <origin xyz="0 0 0.015" rpy="${-pi/2} ${-pi/2} 0"/>
   </joint>
   <!-- Camera frames -->
