Commit message: cleanup codebase - fixing simulation camera

File: vision/urdf/ur30_simple_gripper_camera.urdf.xacro (robot description, xacro)
@@ -130,5 +130,5 @@
         <origin xyz="0 0 0.5" rpy="0 0 0"/>
         <geometry>
-          <!-- FOV: 69° horizontal, depth=1m, width=1.24m, height=0.70m -->
+          <!-- FOV: 69deg horizontal, depth=1m, width=1.24m, height=0.70m -->
           <box size="1.24 0.70 1.0"/>
         </geometry>

File: vision/urdf/ur30_simple_gripper_realsense.urdf.xacro (robot description, xacro)
@@ -58,5 +58,5 @@
     <parent link="gripper_base_link"/>
     <child link="camera_mount_link"/>
-    <origin xyz="0 0.08 0.02" rpy="0 ${pi/6} 0"/>
+    <origin xyz="0 0.08 0.03" rpy="0 ${pi/2} 0"/>
   </joint>
   <!-- RealSense D435i Camera -->
@@ -86,5 +86,5 @@
     <parent link="camera_mount_link"/>
     <child link="camera_link"/>
-    <origin xyz="0 0 0.015" rpy="0 0 0"/>
+    <origin xyz="0 0 0.015" rpy="0 0 ${pi}"/>
   </joint>
   <!-- Camera frames -->
